Commit message: khoa: add mesh and change file path package description

File: ros2/src/myarm_m750_description/urdf/myarm_m750_poe_v3_2.urdf (robot description, URDF)
Before this commit: robot myarm_m750, 11 links, 10 joints
Links:
- link base_link: geometry collision mesh filename=package://myarm_m750_description/urdf/meshes/base_link.dae scale=1 1 1; visual mesh filename=package://myarm_m750_description/urdf/meshes/base_link.dae scale=1 1 1
- link forearm_link: geometry collision mesh filename=package://myarm_m750_description/urdf/meshes/forearm_link.d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 scale=1 1 1; visual mesh filename=package://myarm_m750_description/urdf/meshes/forearm_link.d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 scale=1 1 1
- link gripper_base_link: geometry collision mesh filename=package://myarm_m750_description/urdf/meshes/gripper_base_l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 scale=1 1 1; visual mesh filename=package://myarm_m750_description/urdf/meshes/gripper_base_l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 scale=1 1 1
- link left_gripper_link: geometry collision mesh filename=package://myarm_m750_description/urdf/meshes/left_gripper_l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 scale=1 1 1; visual mesh filename=package://myarm_m750_description/urdf/meshes/left_gripper_l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 scale=1 1 1
- link lower_arm_link: geometry collision mesh filename=package://myarm_m750_description/urdf/meshes/lower_arm_link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 scale=1 1 1; visual mesh filename=package://myarm_m750_description/urdf/meshes/lower_arm_link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 scale=1 1 1
- link right_gripper_link: geometry collision mesh filename=package://myarm_m750_description/urdf/meshes/right_gripper_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 scale=1 1 1; visual mesh filename=package://myarm_m750_description/urdf/meshes/right_gripper_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 scale=1 1 1
- link shoulder_link: geometry collision mesh filename=package://myarm_m750_description/urdf/meshes/shoulder_link.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 scale=1 1 1; visual mesh filename=package://myarm_m750_description/urdf/meshes/shoulder_link.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 scale=1 1 1
- link upper_arm_link: geometry collision mesh filename=package://myarm_m750_description/urdf/meshes/upper_arm_link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 scale=1 1 1; visual mesh filename=package://myarm_m750_description/urdf/meshes/upper_arm_link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 scale=1 1 1
- link wrist_link: geometry collision mesh filename=package://myarm_m750_description/urdf/meshes/wrist_link.dae scale=1 1 1; visual mesh filename=package://myarm_m750_description/urdf/meshes/wrist_link.dae scale=1 1 1
